File: Homematic-6Button-Flush.kicad_pcb (KiCad board)
At the start: 4 copper layers, 50 x 50 mm, 18 parts, among them SW1 SW_Push, SW2 SW_Push, SW3 SW_Push, SW4 SW_Push, SW5 SW_Push, SW6 SW_Push, U1 STM32G030F6Px

Commit message: auto-backup 2026-07-26 08:26:26
Parts:
- moved J_SWD 2.50 mm to (-18.0, -3.50)
Routing:
- net LED_A: track 0.00 -> 9.01 mm, vias 0 -> 1
- net GND: track 0.00 -> 0.62 mm, vias 23 -> 13
- net +3V0: vias 10 -> 6
Changed lines of the file:
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@@
 	(footprint "Connector_PinHeader_2.54mm:PinHeader_1x05_P2.54mm_Vertical"
 		(layer "B.Cu")
-		(at -18 -6)
+		(at -18 -3.5)
 		(descr "Through hole straight pin header, 1x05, 2.54mm pitch, single row")
 		(tags "Through hole pin header THT 1x05 2.54mm single row")
@@
 		(layer "Edge.Cuts")
 	)
+	(segment
+		(start 16 -12.5)
+		(end 15.7 -12.8)
+		(width 0.4)
+		(layer "F.Cu")
+		(net "GND")
+	)
+	(segment
+		(start 15.7 -12.8)
+		(end 15.7 -13)
+		(width 0.4)
+		(layer "F.Cu")
+		(net "GND")
+	)
+	(via
+		(at 15.7 -13)
+		(size 0.5)
+		(drill 0.25)
+		(layers "F.Cu" "B.Cu")
+		(net "GND")
+	)
 	(via
 		(at 2.8625 5.675)
@@
 	)
 	(via
+		(at 0 -11)
+		(size 0.5)
+		(drill 0.25)
+		(layers "F.Cu" "B.Cu")
+		(net "GND")
+	)
+	(via
+		(at 14 11.3)
+		(size 0.5)
+		(drill 0.25)
+		(layers "F.Cu" "B.Cu")
+		(net "GND")
+	)
+	(via
+		(at 14 -1.7)
+		(size 0.5)
+		(drill 0.25)
+		(layers "F.Cu" "B.Cu")
+		(net "GND")
+	)
+	(via
+		(at -6 5.225)
+		(size 0.5)
+		(drill 0.25)
+		(layers "F.Cu" "B.Cu")
+		(net "GND")
+	)
+	(via
+		(at -14 -14.7)
+		(size 0.4)
+		(drill 0.2)
+		(layers "F.Cu" "B.Cu")
+		(net "GND")
+	)
+	(via
+		(at 16 -12.5)
+		(size 0.6)
+		(drill 0.3)
+		(layers "F.Cu" "B.Cu")
+		(net "GND")
+	)
+	(via
+		(at -12.3 0)
+		(size 0.5)
+		(drill 0.25)
+		(layers "F.Cu" "B.Cu")
+		(net "GND")
+	)
+	(via
+		(at -14 11.3)
+		(size 0.4)
+		(drill 0.2)
+		(layers "F.Cu" "B.Cu")
+		(net "GND")
+	)
+	(via
+		(at -0.9375 9)
+		(size 0.5)
+		(drill 0.25)
+		(layers "F.Cu" "B.Cu")
+		(net "GND")
+	)
+	(via
 		(at 6 5.225)
 		(size 0.4)
@@
 	)
 	(via
-		(at 14 11.3)
-		(size 0.5)
-		(drill 0.25)
-		(layers "F.Cu" "B.Cu")
-		(net "GND")
-	)
-	(via
-		(at 6 5.225)
-		(size 0.5)
-		(drill 0.25)
-		(layers "F.Cu" "B.Cu")
-		(net "GND")
-	)
-	(via
-		(at 16 -12.5)
-		(size 0.6)
-		(drill 0.3)
-		(layers "F.Cu" "B.Cu")
-		(net "GND")
-	)
-	(via
-		(at 14 -1.7)
-		(size 0.5)
-		(drill 0.25)
-		(layers "F.Cu" "B.Cu")
-		(net "GND")
-	)
-	(via
-		(at -6 5.225)
-		(size 0.5)
-		(drill 0.25)
-		(layers "F.Cu" "B.Cu")
-		(net "GND")
-	)
-	(via
-		(at -14 -14.7)
-		(size 0.4)
-		(drill 0.2)
-		(layers "F.Cu" "B.Cu")
-		(net "GND")
-	)
-	(via
-		(at -12.3 0)
-		(size 0.5)
-		(drill 0.25)
-		(layers "F.Cu" "B.Cu")
-		(net "GND")
-	)
-	(via
-		(at -14 11.3)
-		(size 0.4)
-		(drill 0.2)
-		(layers "F.Cu" "B.Cu")
-		(net "GND")
-	)
-	(via
-		(at 0 -11)
-		(size 0.5)
-		(drill 0.25)
-		(layers "F.Cu" "B.Cu")
-		(net "GND")
-	)
-	(via
-		(at 15.7 -13)
-		(size 0.5)
-		(drill 0.25)
-		(layers "F.Cu" "B.Cu")
-		(net "GND")
-	)
-	(via
-		(at -12.3 0)
-		(size 0.4)
-		(drill 0.2)
-		(layers "F.Cu" "B.Cu")
-		(net "GND")
-	)
-	(via
-		(at -0.9375 9)
-		(size 0.5)
-		(drill 0.25)
-		(layers "F.Cu" "B.Cu")
-		(net "GND")
-	)
-	(via
-		(at -14 11.3)
-		(size 0.5)
-		(drill 0.25)
-		(layers "F.Cu" "B.Cu")
-		(net "GND")
-	)
-	(via
 		(at 11.05 3)
 		(size 0.5)
@@
 		(net "GND")
 	)
-	(via
-		(at 11.05 3)
-		(size 0.4)
-		(drill 0.2)
-		(layers "F.Cu" "B.Cu")
-		(net "GND")
-	)
-	(via
-		(at 0 -11)
+	(segment
+		(start 0.9647 10.6429)
+		(end 0.9375 10.6157)
+		(width 0.4)
+		(layer "F.Cu")
+		(net "LED_A")
+	)
+	(segment
+		(start 0.9375 10.6157)
+		(end 0.9375 9)
+		(width 0.4)
+		(layer "F.Cu")
+		(net "LED_A")
+	)
+	(via
+		(at 0.9647 10.6429)
 		(size 0.6)
 		(drill 0.3)
 		(layers "F.Cu" "B.Cu")
-		(net "GND")
-	)
-	(via
-		(at 14 -1.7)
-		(size 0.4)
-		(drill 0.2)
-		(layers "F.Cu" "B.Cu")
-		(net "GND")
-	)
-	(via
-		(at -14 -14.7)
-		(size 0.5)
-		(drill 0.25)
-		(layers "F.Cu" "B.Cu")
-		(net "GND")
-	)
-	(via
-		(at -6 5.225)
-		(size 0.4)
-		(drill 0.2)
-		(layers "F.Cu" "B.Cu")
-		(net "GND")
-	)
-	(via
-		(at -0.9375 9)
-		(size 0.4)
-		(drill 0.2)
-		(layers "F.Cu" "B.Cu")
-		(net "GND")
-	)
-	(via
-		(at 14 11.3)
-		(size 0.4)
-		(drill 0.2)
-		(layers "F.Cu" "B.Cu")
-		(net "GND")
+		(net "LED_A")
+	)
+	(segment
+		(start 1.3218 11)
+		(end 0.9647 10.6429)
+		(width 0.4)
+		(layer "B.Cu")
+		(net "LED_A")
+	)
+	(segment
+		(start 8.175 11)
+		(end 1.3218 11)
+		(width 0.4)
+		(layer "B.Cu")
+		(net "LED_A")
 	)
 	(via
@@
 	)
 	(via
+		(at -12.8 -11)
+		(size 0.5)
+		(drill 0.25)
+		(layers "F.Cu" "B.Cu")
+		(net "+3V0")
+	)
+	(via
+		(at 12.8 -11)
+		(size 0.5)
+		(drill 0.25)
+		(layers "F.Cu" "B.Cu")
+		(net "+3V0")
+	)
+	(via
+		(at -6 6.775)
+		(size 0.5)
+		(drill 0.25)
+		(layers "F.Cu" "B.Cu")
+		(net "+3V0")
+	)
+	(via
 		(at 12.95 3)
 		(size 0.5)
 		(drill 0.25)
-		(layers "F.Cu" "B.Cu")
-		(net "+3V0")
-	)
-	(via
-		(at -6 6.775)
-		(size 0.5)
-		(drill 0.25)
-		(layers "F.Cu" "B.Cu")
-		(net "+3V0")
-	)
-	(via
-		(at -6 6.775)
-		(size 0.4)
-		(drill 0.2)
-		(layers "F.Cu" "B.Cu")
-		(net "+3V0")
-	)
-	(via
-		(at 12.8 -11)
-		(size 0.5)
-		(drill 0.25)
-		(layers "F.Cu" "B.Cu")
-		(net "+3V0")
-	)
-	(via
-		(at 12.95 3)
-		(size 0.4)
-		(drill 0.2)
-		(layers "F.Cu" "B.Cu")
-		(net "+3V0")
-	)
-	(via
-		(at -12.8 -11)
-		(size 0.5)
-		(drill 0.25)
-		(layers "F.Cu" "B.Cu")
-		(net "+3V0")
-	)
-	(via
-		(at 12.8 -11)
-		(size 0.6)
-		(drill 0.3)
-		(layers "F.Cu" "B.Cu")
-		(net "+3V0")
-	)
-	(via
-		(at 6 6.775)
-		(size 0.5)
-		(drill 0.25)

Commit message: auto-backup 2026-07-26 09:26:22
Parts:
- moved SW1 1.50 mm to (-15.1, 14.0)
- moved SW3 1.50 mm to (-15.1, -14.0)
- moved SW4 1.50 mm to (15.1, 14.0)
- moved SW6 1.50 mm to (15.1, -14.0)
- moved SW2 1.50 mm to (-15.5, 0.00)
- moved SW5 1.50 mm to (15.5, 0.00)
- moved J_RF 1.20 mm to (9.00, 15.2)
- moved J_SWD 0.60 mm to (-18.6, -3.50)
Routing:
- net BTN1: track 0.00 -> 38.1 mm, vias 0 -> 1
- net BTN5: track 0.00 -> 35.9 mm, vias 0 -> 1
- net BTN3: track 0.00 -> 34.7 mm, vias 0 -> 1
- net BTN6: track 0.00 -> 31.1 mm, vias 0 -> 1
- net NRST: track 0.00 -> 30.9 mm
- net BTN2: track 0.00 -> 24.1 mm, vias 0 -> 1
- net RF_GDO2: track 0.00 -> 23.6 mm, vias 0 -> 1
- net SWCLK: track 0.00 -> 21.2 mm
- net SWDIO: track 0.00 -> 20.1 mm
- net LED_CTRL: track 0.00 -> 17.6 mm
- net SPI_MOSI: track 0.00 -> 17.3 mm, vias 0 -> 1
- net BTN4: track 0.00 -> 15.7 mm, vias 0 -> 1
- net RF_GDO0: track 0.00 -> 13.8 mm, vias 0 -> 1
- net RF_CSN: track 0.00 -> 11.6 mm
- net SPI_SCK: track 0.00 -> 11.5 mm
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